File: knock_sensor.sch (EAGLE design)
At the start: 19 parts, among them IC1 7805T, U1 TLC2262CP

Commit message: Needs to be finished
Connections:
- removed net PIEZO: U1.1IN+
- net ECU_IN: now also SV1.3
- net ECU_OUT: now also SV1.2
- net GND: now also SV1.4
- net N$2: now also SV1.1, U1.1IN+; no longer C6.2, ZU4.AVCC, ZU4.VCC
- net VCC: now also C6.2, SV1.5, ZU4.AVCC, ZU4.VCC; no longer IC1.VO, R2.1
Other:
- moved on the sheet: C4, JP5
